Commit message: Continued working on urdf, cases and bases complete (visuals)

File: software/urdf/qutee.urdf (robot description, URDF)
Before this commit: robot qutee_robot, 3 links, 2 joints
Links:
- added link bottom_case_link; visual box size=0.003 0.057 0.0082; visual box size=0.003 0.057 0.0082
- added link top_case_link; visual box size=0.0021 0.0544 0.002; visual box size=0.0085 0.0544 0.0055
Joints:
- added joint body_base_sq_top_case_joint: type fixed, parent body_base_sq_link, child top_case_link, origin xyz=0 0 0.01055 rpy=0 0 0
- added joint body_bottom_sq_bottom_case_joint: type fixed, parent body_bottom_sq_link, child bottom_case_link, origin xyz=0 0 -0.0089 rpy=0 0 0

Commit message: continuing working on urdf, working on doubleU links

File: software/urdf/qutee.urdf (robot description, URDF)
Before this commit: robot qutee_robot, 5 links, 4 joints
Links:
- added link front_doubleu_link; visual cylinder length=0.0022 radius=0.01
- added link front_motor_link; visual box size=0.034 0.02 0.023
- added link left_motor_link; visual box size=0.02 0.034 0.023
- added link rear_motor_link; visual box size=0.034 0.02 0.023
- added link right_motor_link; visual box size=0.02 0.034 0.023
Joints:
- added joint body_base_sq_front_motor_joint: type fixed, parent body_base_sq_link, child front_motor_link, origin xyz=0.0355 0 -0.013 rpy=0 0 0
- added joint body_base_sq_left_motor_joint: type fixed, parent body_base_sq_link, child left_motor_link, origin xyz=0 0.0355 -0.013 rpy=0 0 0
- added joint body_base_sq_rear_motor_joint: type fixed, parent body_base_sq_link, child rear_motor_link, origin xyz=-0.0355 0 -0.013 rpy=0 0 0
- added joint body_base_sq_right_motor_joint: type fixed, parent body_base_sq_link, child right_motor_link, origin xyz=0 -0.0355 -0.013 rpy=0 0 0
- added joint front_motor_front_doubleu_joint: type continuous, parent front_motor_link, child front_doubleu_link, origin xyz=0.0075 0 0.0115 rpy=0 0 0, axis 0 0 1

Commit message: still working on doubleu links

File: software/urdf/qutee.urdf (robot description, URDF)
Before this commit: robot qutee_robot, 10 links, 9 joints
Links:
- link front_doubleu_link: geometry visual box size=0.0022 0.02 0.0334; visual box size=0.0022 0.0334 0.02
Joints:
- joint front_motor_front_doubleu_joint: origin xyz=0.0075 0 0.0115 rpy=0 0 0 -> xyz=0.0075 0 0.013 rpy=0 0 0

Commit message: urdf thighs and motors complete (visuals only), still to add legs

File: software/urdf/qutee.urdf (robot description, URDF)
Before this commit: robot qutee_robot, 10 links, 9 joints
Links:
- removed link front_motor_link
- removed link left_motor_link
- removed link rear_motor_link
- removed link right_motor_link
- added link front_body_motor_link; visual box size=0.034 0.02 0.023
- added link front_leg_motor_link; visual box size=0.034 0.023 0.02
- added link front_side_link; visual box size=0.072 0.0022 0.02; visual box size=0.072 0.0022 0.02
- added link front_thigh_motor_link; visual box size=0.034 0.023 0.02
- added link left_body_motor_link; visual box size=0.02 0.034 0.023
- added link left_doubleu_link; visual box size=0.0022 0.0181 0.02; visual box size=0.0022 0.0181 0.02
- added link left_leg_motor_link; visual box size=0.023 0.034 0.02
- added link left_side_link; visual box size=0.0022 0.072 0.02; visual box size=0.0022 0.072 0.02
- added link left_thigh_motor_link; visual box size=0.023 0.034 0.02
- added link rear_body_motor_link; visual box size=0.034 0.02 0.023
- added link rear_doubleu_link; visual box size=0.0022 0.02 0.0334; visual box size=0.0022 0.0334 0.02
- added link rear_leg_motor_link; visual box size=0.034 0.023 0.02
- added link rear_side_link; visual box size=0.072 0.0022 0.02; visual box size=0.072 0.0022 0.02
- added link rear_thigh_motor_link; visual box size=0.034 0.023 0.02
- added link right_body_motor_link; visual box size=0.02 0.034 0.023
- added link right_doubleu_link; visual box size=0.0022 0.0181 0.02; visual box size=0.0022 0.0181 0.02
- added link right_leg_motor_link; visual box size=0.023 0.034 0.02
- added link right_side_link; visual box size=0.0022 0.072 0.02; visual box size=0.0022 0.072 0.02
- added link right_thigh_motor_link; visual box size=0.023 0.034 0.02
- link front_doubleu_link: geometry visual box size=0.0022 0.02 0.0334; visual box size=0.0022 0.0334 0.02
Joints:
- removed joint body_base_sq_front_motor_joint
- removed joint body_base_sq_left_motor_joint
- removed joint body_base_sq_rear_motor_joint
- removed joint body_base_sq_right_motor_joint
- removed joint front_motor_front_doubleu_joint
- added joint body_base_sq_front_body_motor_joint: type fixed, parent body_base_sq_link, child front_body_motor_link, origin xyz=0.0355 0 -0.013 rpy=0 0 0
- added joint body_base_sq_left_body_motor_joint: type fixed, parent body_base_sq_link, child left_body_motor_link, origin xyz=0 0.0355 -0.013 rpy=0 0 0
- added joint body_base_sq_rear_body_motor_joint: type fixed, parent body_base_sq_link, child rear_body_motor_link, origin xyz=-0.0355 0 -0.013 rpy=0 0 0
- added joint body_base_sq_right_body_motor_joint: type fixed, parent body_base_sq_link, child right_body_motor_link, origin xyz=0 -0.0355 -0.013 rpy=0 0 0
- added joint front_body_motor_front_doubleu_joint: type continuous, parent front_body_motor_link, child front_doubleu_link, origin xyz=0.0075 0 0.013 rpy=0 0 0, axis 0 0 -1
- added joint front_doubleu_front_thigh_motor_joint: type continuous, parent front_doubleu_link, child front_thigh_motor_link, origin xyz=0.0362 -0.0156 -0.013 rpy=0 0 0, axis 0 1 0
- added joint front_side_front_leg_motor_joint: type fixed, parent front_side_link, child front_leg_motor_link, origin xyz=0.018 0 0 rpy=0 0 0
- added joint front_thigh_motor_front_side_joint: type fixed, parent front_thigh_motor_link, child front_side_link, origin xyz=0.0255 0.0156 0 rpy=0 0 0
- added joint left_body_motor_left_doubleu_joint: type continuous, parent left_body_motor_link, child left_doubleu_link, origin xyz=0 0.0075 0.013 rpy=0 0 0, axis 0 0 -1
- added joint left_doubleu_left_thigh_motor_joint: type continuous, parent left_doubleu_link, child left_thigh_motor_link, origin xyz=-0.0156 0.0362 -0.013 rpy=0 0 0, axis -1 0 0
- added joint left_side_left_leg_motor_joint: type fixed, parent left_side_link, child left_leg_motor_link, origin xyz=0 0.018 0 rpy=0 0 0
- added joint left_thigh_motor_left_side_joint: type fixed, parent left_thigh_motor_link, child left_side_link, origin xyz=0.0156 0.0255 0 rpy=0 0 0
- added joint rear_body_motor_rear_doubleu_joint: type continuous, parent rear_body_motor_link, child rear_doubleu_link, origin xyz=-0.0075 0 0.013 rpy=0 0 0, axis 0 0 -1
- added joint rear_doubleu_rear_thigh_motor_joint: type continuous, parent rear_doubleu_link, child rear_thigh_motor_link, origin xyz=-0.0362 -0.0156 -0.013 rpy=0 0 0, axis 0 -1 0
- added joint rear_side_rear_leg_motor_joint: type fixed, parent rear_side_link, child rear_leg_motor_link, origin xyz=-0.018 0 0 rpy=0 0 0
- added joint rear_thigh_motor_rear_side_joint: type fixed, parent rear_thigh_motor_link, child rear_side_link, origin xyz=-0.0255 0.0156 0 rpy=0 0 0
- added joint right_body_motor_right_doubleu_joint: type continuous, parent right_body_motor_link, child right_doubleu_link, origin xyz=0 -0.0075 0.013 rpy=0 0 0, axis 0 0 -1
- added joint right_doubleu_right_thigh_motor_joint: type continuous, parent right_doubleu_link, child right_thigh_motor_link, origin xyz=-0.0156 -0.0362 -0.013 rpy=0 0 0, axis 1 0 0
- added joint right_side_right_leg_motor_joint: type fixed, parent right_side_link, child right_leg_motor_link, origin xyz=0 -0.018 0 rpy=0 0 0
- added joint right_thigh_motor_right_side_joint: type fixed, parent right_thigh_motor_link, child right_side_link, origin xyz=0.0156 -0.0255 0 rpy=0 0 0

Commit message: urdf visuals finished

File: software/urdf/qutee.urdf (robot description, URDF)
Before this commit: robot qutee_robot, 25 links, 24 joints
Links:
- added link front_leg_link; visual box size=0.005 0.0022 0.0247; visual box size=0.005 0.0022 0.0247
- added link left_leg_link; visual box size=0.0022 0.005 0.0247; visual box size=0.0022 0.005 0.0247
- added link rear_leg_link; visual box size=0.005 0.0022 0.0247; visual box size=0.005 0.0022 0.0247
- added link right_leg_link; visual box size=0.0022 0.005 0.0247; visual box size=0.0022 0.005 0.0247
Joints:
- added joint front_leg_motor_front_leg_joint: type continuous, parent front_leg_motor_link, child front_leg_link, origin xyz=0.0075 -0.0126 0 rpy=0 0 0, axis 0 1 0
- added joint left_leg_motor_left_leg_joint: type continuous, parent left_leg_motor_link, child left_leg_link, origin xyz=-0.0126 0.0075 0 rpy=0 0 0, axis -1 0 0
- added joint rear_leg_motor_rear_leg_joint: type continuous, parent rear_leg_motor_link, child rear_leg_link, origin xyz=-0.0075 -0.0126 0 rpy=0 0 0, axis 0 -1 0
- added joint right_leg_motor_right_leg_joint: type continuous, parent right_leg_motor_link, child right_leg_link, origin xyz=-0.0126 -0.0075 0 rpy=0 0 0, axis 1 0 0

Commit message: collision and inertial tags added to urdf

File: software/urdf/qutee.urdf (robot description, URDF)
Before this commit: robot qutee_robot, 29 links, 28 joints
Links:
- added link base_footprint_link
- added link front_dummy_leg_diag1_link; collision box size=0.02 0.0022 0.0207; visual box size=0 0 0
- added link front_dummy_leg_diag2_link; collision box size=0.02 0.0022 0.0207; visual box size=0 0 0
- added link front_dummy_leg_low_horiz_link; collision box size=0.02 0.0099 0.0022; visual box size=0 0 0
- added link front_dummy_leg_mid_horiz_link; collision box size=0.02 0.03715 0.0139; visual box size=0 0 0
- added link left_dummy_leg_diag1_link; collision box size=0.0022 0.02 0.0207; visual box size=0 0 0
- added link left_dummy_leg_diag2_link; collision box size=0.0022 0.02 0.0207; visual box size=0 0 0
- added link left_dummy_leg_low_horiz_link; collision box size=0.0099 0.02 0.0022; visual box size=0 0 0
- added link left_dummy_leg_mid_horiz_link; collision box size=0.03715 0.02 0.0139; visual box size=0 0 0
- added link rear_dummy_leg_diag1_link; collision box size=0.02 0.0022 0.0207; visual box size=0 0 0
- added link rear_dummy_leg_diag2_link; collision box size=0.02 0.0022 0.0207; visual box size=0 0 0
- added link rear_dummy_leg_low_horiz_link; collision box size=0.02 0.0099 0.0022; visual box size=0 0 0
- added link rear_dummy_leg_mid_horiz_link; collision box size=0.02 0.03715 0.0139; visual box size=0 0 0
- added link right_dummy_leg_diag1_link; collision box size=0.0022 0.02 0.0207; visual box size=0 0 0
- added link right_dummy_leg_diag2_link; collision box size=0.0022 0.02 0.0207; visual box size=0 0 0
- added link right_dummy_leg_low_horiz_link; collision box size=0.0099 0.02 0.0022; visual box size=0 0 0
- added link right_dummy_leg_mid_horiz_link; collision box size=0.03715 0.02 0.0139; visual box size=0 0 0
- added link world_link
- link base_link: mass None -> 0.28667; geometry collision box size=0.035 0.034 0.03; visual box size=0.035 0.034 0.03
- link body_base_sq_link: mass None -> 0.09567; geometry collision box size=0.0888 0.0888 0.002; visual box size=0.078 0.078 0.002
- link body_bottom_sq_link: mass None -> 0.09567; geometry collision box size=0.0888 0.0888 0.002; visual box size=0.078 0.078 0.002
- link bottom_case_link: mass None -> 0.08877; geometry collision box size=0.08 0.0741 0.0237; visual box size=0.003 0.057 0.0082
- link front_body_motor_link: mass None -> 0.12454; geometry collision box size=0.034 0.02 0.023; visual box size=0.034 0.02 0.023
- link front_doubleu_link: mass None -> 0.0439; geometry collision box size=0.0562 0.0334 0.0334; visual box size=0.0022 0.02 0.0334
- link front_leg_link: mass None -> 0.13034; geometry collision box size=0.02 0.0334 0.1052; visual box size=0.005 0.0022 0.0247
- link front_leg_motor_link: mass None -> 0.12454; geometry collision box size=0.034 0.023 0.02; visual box size=0.034 0.023 0.02
- link front_side_link: mass None -> 0.0372; geometry collision box size=0.072 0.0274 0.02; visual box size=0.072 0.0022 0.02
- link front_thigh_motor_link: mass None -> 0.12454; geometry collision box size=0.034 0.023 0.02; visual box size=0.034 0.023 0.02
- link left_body_motor_link: mass None -> 0.12454; geometry collision box size=0.02 0.034 0.023; visual box size=0.02 0.034 0.023
- link left_doubleu_link: mass None -> 0.0439; geometry collision box size=0.0334 0.0562 0.0334; visual box size=0.0022 0.0181 0.02
- link left_leg_link: mass None -> 0.13034; geometry collision box size=0.0334 0.02 0.1052; visual box size=0.0022 0.005 0.0247
- link left_leg_motor_link: mass None -> 0.12454; geometry collision box size=0.023 0.034 0.02; visual box size=0.023 0.034 0.02
- link left_side_link: mass None -> 0.0372; geometry collision box size=0.0274 0.072 0.02; visual box size=0.0022 0.072 0.02
- link left_thigh_motor_link: mass None -> 0.12454; geometry collision box size=0.023 0.034 0.02; visual box size=0.023 0.034 0.02
- link rear_body_motor_link: mass None -> 0.12454; geometry collision box size=0.034 0.02 0.023; visual box size=0.034 0.02 0.023
- link rear_doubleu_link: mass None -> 0.0439; geometry collision box size=0.0562 0.0334 0.0334; visual box size=0.0022 0.02 0.0334
- link rear_leg_link: mass None -> 0.13034; geometry collision box size=0.02 0.0334 0.1052; visual box size=0.005 0.0022 0.0247
- link rear_leg_motor_link: mass None -> 0.12454; geometry collision box size=0.034 0.023 0.02; visual box size=0.034 0.023 0.02
- link rear_side_link: mass None -> 0.0372; geometry collision box size=0.072 0.0274 0.02; visual box size=0.072 0.0022 0.02
- link rear_thigh_motor_link: mass None -> 0.12454; geometry collision box size=0.034 0.023 0.02; visual box size=0.034 0.023 0.02
- link right_body_motor_link: mass None -> 0.12454; geometry collision box size=0.02 0.034 0.023; visual box size=0.02 0.034 0.023
- link right_doubleu_link: mass None -> 0.0439; geometry collision box size=0.0334 0.0562 0.0334; visual box size=0.0022 0.0181 0.02
- link right_leg_link: mass None -> 0.13034; geometry collision box size=0.0334 0.02 0.1052; visual box size=0.0022 0.005 0.0247
- link right_leg_motor_link: mass None -> 0.12454; geometry collision box size=0.023 0.034 0.02; visual box size=0.023 0.034 0.02
- link right_side_link: mass None -> 0.0372; geometry collision box size=0.0274 0.072 0.02; visual box size=0.0022 0.072 0.02
- link right_thigh_motor_link: mass None -> 0.12454; geometry collision box size=0.023 0.034 0.02; visual box size=0.023 0.034 0.02
- link top_case_link: mass None -> 0.17261; geometry collision box size=0.08 0.0741 0.0237; visual box size=0.0021 0.0544 0.002
Joints:
- added joint base_joint: type fixed, parent base_footprint_link, child base_link, origin xyz=0 0 0 rpy=0 0 0
- added joint front_leg_front_dummy_leg_diag1_joint: type fixed, parent front_leg_link, child front_dummy_leg_diag1_link, origin xyz=0 0 0 rpy=0 0 0
- added joint front_leg_front_dummy_leg_diag2_joint: type fixed, parent front_leg_link, child front_dummy_leg_diag2_link, origin xyz=0 0 0 rpy=0 0 0
- added joint front_leg_front_dummy_leg_mid_horiz_joint: type fixed, parent front_leg_link, child front_dummy_leg_mid_horiz_link, origin xyz=0 0 0 rpy=0 0 0
- added joint front_leg_front_dummy_low_horiz_joint: type fixed, parent front_leg_link, child front_dummy_leg_low_horiz_link, origin xyz=0 0 0 rpy=0 0 0
- added joint left_leg_left_dummy_leg_diag1_joint: type fixed, parent left_leg_link, child left_dummy_leg_diag1_link, origin xyz=0 0 0 rpy=0 0 0
- added joint left_leg_left_dummy_leg_diag2_joint: type fixed, parent left_leg_link, child left_dummy_leg_diag2_link, origin xyz=0 0 0 rpy=0 0 0
- added joint left_leg_left_dummy_leg_mid_horiz_joint: type fixed, parent left_leg_link, child left_dummy_leg_mid_horiz_link, origin xyz=0 0 0 rpy=0 0 0
- added joint left_leg_left_dummy_low_horiz_joint: type fixed, parent left_leg_link, child left_dummy_leg_low_horiz_link, origin xyz=0 0 0 rpy=0 0 0
- added joint rear_leg_rear_dummy_leg_diag1_joint: type fixed, parent rear_leg_link, child rear_dummy_leg_diag1_link, origin xyz=0 0 0 rpy=0 0 0
- added joint rear_leg_rear_dummy_leg_diag2_joint: type fixed, parent rear_leg_link, child rear_dummy_leg_diag2_link, origin xyz=0 0 0 rpy=0 0 0
- added joint rear_leg_rear_dummy_leg_mid_horiz_joint: type fixed, parent rear_leg_link, child rear_dummy_leg_mid_horiz_link, origin xyz=0 0 0 rpy=0 0 0
- added joint rear_leg_rear_dummy_low_horiz_joint: type fixed, parent rear_leg_link, child rear_dummy_leg_low_horiz_link, origin xyz=0 0 0 rpy=0 0 0
- added joint right_leg_right_dummy_leg_diag1_joint: type fixed, parent right_leg_link, child right_dummy_leg_diag1_link, origin xyz=0 0 0 rpy=0 0 0
- added joint right_leg_right_dummy_leg_diag2_joint: type fixed, parent right_leg_link, child right_dummy_leg_diag2_link, origin xyz=0 0 0 rpy=0 0 0
- added joint right_leg_right_dummy_leg_mid_horiz_joint: type fixed, parent right_leg_link, child right_dummy_leg_mid_horiz_link, origin xyz=0 0 0 rpy=0 0 0
- added joint right_leg_right_dummy_low_horiz_joint: type fixed, parent right_leg_link, child right_dummy_leg_low_horiz_link, origin xyz=0 0 0 rpy=0 0 0
- added joint world_base_footprint_joint: type fixed, parent world_link, child base_footprint_link, origin xyz=0 0 0 rpy=0 0 0

Commit message: Joints changed to revolute

File: software/urdf/qutee.urdf (robot description, URDF)
Before this commit: robot qutee_robot, 47 links, 46 joints
Joints:
- joint front_body_motor_front_doubleu_joint: limit (none) -> lower=-1.5708 upper=1.5708 effort=10.0 velocity=10.0; type continuous -> revolute
- joint front_doubleu_front_thigh_motor_joint: limit (none) -> lower=-1.9199 upper=1.9199 effort=10.0 velocity=10.0; type continuous -> revolute
- joint front_leg_motor_front_leg_joint: limit (none) -> lower=-4.18879 upper=1.0472 effort=10.0 velocity=10.0; type continuous -> revolute
- joint left_body_motor_left_doubleu_joint: limit (none) -> lower=-1.5708 upper=1.5708 effort=10.0 velocity=10.0; type continuous -> revolute
- joint left_doubleu_left_thigh_motor_joint: limit (none) -> lower=-1.9199 upper=1.9199 effort=10.0 velocity=10.0; type continuous -> revolute
- joint left_leg_motor_left_leg_joint: limit (none) -> lower=-4.18879 upper=1.0472 effort=10.0 velocity=10.0; type continuous -> revolute
- joint rear_body_motor_rear_doubleu_joint: limit (none) -> lower=-1.5708 upper=1.5708 effort=10.0 velocity=10.0; type continuous -> revolute
- joint rear_doubleu_rear_thigh_motor_joint: limit (none) -> lower=-1.9199 upper=1.9199 effort=10.0 velocity=10.0; type continuous -> revolute
- joint rear_leg_motor_rear_leg_joint: limit (none) -> lower=-4.18879 upper=1.0472 effort=10.0 velocity=10.0; type continuous -> revolute
- joint right_body_motor_right_doubleu_joint: limit (none) -> lower=-1.5708 upper=1.5708 effort=10.0 velocity=10.0; type continuous -> revolute
- joint right_doubleu_right_thigh_motor_joint: limit (none) -> lower=-1.9199 upper=1.9199 effort=10.0 velocity=10.0; type continuous -> revolute
- joint right_leg_motor_right_leg_joint: limit (none) -> lower=-4.18879 upper=1.0472 effort=10.0 velocity=10.0; type continuous -> revolute
